Commit message: add sensor and laser scan

File: my_robot/urdf/my_robot.xacro (robot description, xacro)
@@ -1,4 +1,5 @@
 <?xml version='1.0'?>
 <robot name="my_robot" xmlns:xacro="http://www.ros.org/wiki/xacro">
+  <xacro:include filename="$(find my_robot)/urdf/my_robot.gazebo"/>
   <link name="robot_footprint"></link>
   <joint name="robot_footprint_joint" type="fixed">
@@ -117,3 +118,61 @@
     <dynamics damping="1.0" friction="1.0"/>
   </joint>
+   <link name="camera">
+     <visual name="visual_camera">
+       <origin xyz="0 0 0" rpy="0 0 0"/>
+         <geometry>
+           <box size="0.05 0.05 0.05"/>
+         </geometry>
+     </visual>
+     <collision name="collision_camera">
+         <origin xyz="0 0 0" rpy="0 0 0"/>
+            <geometry>
+              <box size="0.05 0.05 0.05"/>
+         </geometry>
+     </collision>
+     <inertial>
+       <mass value="0.1"/>
+       <origin xyz="0 0 0" rpy=" 0 0 0"/>
+       <inertia
+          ixx="0.1" ixy="0" ixz="0"
+          iyy="0.1" iyz="0"
+          izz="0.1"
+      />
+     </inertial>
+   </link>
+    <joint type="fixed" name="camera_joint">
+      <origin xyz="0.2 0 0" rpy="0 0 0"/>
+      <child link="camera"/>
+      <parent link="chassis"/>
+      <axis xyz="0 1 0" rpy="0 0 0"/>
+    </joint>
+  <link name="hokuyo">
+     <visual name="visual_hokuyo">
+       <origin xyz="0 0 0" rpy="0 0 0"/>
+         <geometry>
+           <mesh filename="package://my_robot/meshes/hokuyo.dae"/>
+         </geometry>
+     </visual>
+     <collision name="collision_hokuyo">
+         <origin xyz="0 0 0" rpy="0 0 0"/>
+            <geometry>
+              <box size="0.1 0.1 0.1"/>
+         </geometry>
+     </collision>
+     <inertial>
+       <mass value="0.1"/>
+       <origin xyz="0 0 0" rpy=" 0 0 0"/>
+       <inertia
+          ixx="0.000001" ixy="0" ixz="0"
+          iyy="0.000001" iyz="0"
+          izz="0.000001"
+      />
+     </inertial>
+   </link>
+    <joint type="fixed" name="hokuyo_joint">
+      <origin xyz="0.15 0 0.1" rpy="0 0 0"/>
+      <child link="hokuyo"/>
+      <parent link="chassis"/>
+      <axis xyz="0 1 0" rpy="0 0 0"/>
+    </joint>
 </robot>
